Commit message: fix joint axis

File: rm_description/urdf/mount.urdf.xacro (robot description, xacro)
@@ -27,5 +27,5 @@
 	</joint>
 	<joint name="servo_joint" type="revolute">
-		<axis xyz="0 -1 0"/>
+		<axis xyz="0 1 0"/>
 		<limit lower="${-M_PI/4}" upper="${M_PI/4}" effort="10" velocity="10"/>
 		<origin xyz="0 0.0035 0.325" rpy="0 0 0"/>
